Commit message: map_inner

File: unitree_gazebo/urdf/terrain/terrainmap1.urdf.xacro (robot description, xacro)
@@ -6,9 +6,6 @@
 	<link name="world"/>
 	<xacro:include filename="$(find unitree_gazebo)/urdf/obstacles/materials.xacro" />
-	<!-- Terrain 1,2,3,4,6
+	<!-- Terrain 1,2,3,4,6 -->
 	<xacro:include filename="$(find unitree_gazebo)/urdf/test/terrain_inner.urdf.xacro"/>
 	<xacro:terrain_inner parent="world" handle="1" position="+4.7692e-01 +2.3249e-01 +2.9749e-01" orientation="0 0 0"/> -->
-	<!-- Terrain 1 -->
-	<xacro:include filename="$(find unitree_gazebo)/urdf/test/terrain1_inner.urdf.xacro"/>
-	<xacro:terrain1_inner parent="world" handle="1" position="+4.3601e+00 +1.2215e+00 +2.9750e-01" orientation="0 0 0"/>
 </robot>

File: unitree_gazebo/urdf/terrain/terrainmap3.urdf (robot description, URDF)
Before this commit: robot competition_map_inner, 2 links, 1 joints
Links:
- removed link terrain1_inner_1
- added link terrain_inner_1, mass 1; collision mesh filename=package://unitree_gazebo/meshes/compound/terrain_inner.stl; visual mesh filename=package://unitree_gazebo/meshes/compound/terrain_inner.stl
Joints:
- removed joint terrain1_inner_1_joint
- added joint terrain_inner_1_joint: type fixed, parent world, child terrain_inner_1, origin xyz=+4.7692e-01 +2.3249e-01 +2.9749e-01 rpy=0 0 0
