Commit message: add vel

File: robots/aliengo_description/urdf/aliengo.urdf (robot description, URDF)
Before this commit: robot aliengo, 31 links, 30 joints
Links:
- removed link FL_calf_rotor
- removed link FL_hip_rotor
- removed link FL_thigh_rotor
- removed link FR_calf_rotor
- removed link FR_hip_rotor
- removed link FR_thigh_rotor
- removed link RL_calf_rotor
- removed link RL_hip_rotor
- removed link RL_thigh_rotor
- removed link RR_calf_rotor
- removed link RR_hip_rotor
- removed link RR_thigh_rotor
- link FL_calf: geometry collision box size=0.25 0.0208 0.016; visual mesh filename=../meshes/calf.dae scale=1 1 1
- link FL_hip: geometry collision cylinder length=0.0418 radius=0.046; visual mesh filename=../meshes/hip.dae scale=1 1 1
- link FL_thigh: geometry collision box size=0.25 0.0374 0.043; visual mesh filename=../meshes/thigh.dae scale=1 1 1
- link FR_calf: geometry collision box size=0.25 0.0208 0.016; visual mesh filename=../meshes/calf.dae scale=1 1 1
- link FR_hip: geometry collision cylinder length=0.0418 radius=0.046; visual mesh filename=../meshes/hip.dae scale=1 1 1
- link FR_thigh: geometry collision box size=0.25 0.0374 0.043; visual mesh filename=../meshes/thigh_mirror.dae scale=1 1 1
- link RL_calf: geometry collision box size=0.25 0.0208 0.016; visual mesh filename=../meshes/calf.dae scale=1 1 1
- link RL_hip: geometry collision cylinder length=0.0418 radius=0.046; visual mesh filename=../meshes/hip.dae scale=1 1 1
- link RL_thigh: geometry collision box size=0.25 0.0374 0.043; visual mesh filename=../meshes/thigh.dae scale=1 1 1
- link RR_calf: geometry collision box size=0.25 0.0208 0.016; visual mesh filename=../meshes/calf.dae scale=1 1 1
- link RR_hip: geometry collision cylinder length=0.0418 radius=0.046; visual mesh filename=../meshes/hip.dae scale=1 1 1
- link RR_thigh: geometry collision box size=0.25 0.0374 0.043; visual mesh filename=../meshes/thigh_mirror.dae scale=1 1 1
- link trunk: mass 11.644 -> 9.041; geometry collision box size=0.647 0.15 0.112; visual mesh filename=../meshes/trunk.dae scale=1 1 1
Joints:
- removed joint FL_calf_rotor_joint
- removed joint FL_hip_rotor_joint
- removed joint FL_thigh_rotor_joint
- removed joint FR_calf_rotor_joint
- removed joint FR_hip_rotor_joint
- removed joint FR_thigh_rotor_joint
- removed joint RL_calf_rotor_joint
- removed joint RL_hip_rotor_joint
- removed joint RL_thigh_rotor_joint
- removed joint RR_calf_rotor_joint
- removed joint RR_hip_rotor_joint
- removed joint RR_thigh_rotor_joint
- joint FL_calf_joint: limit lower=-2.775073510670984 upper=-0.6457718232379019 effort=44.4 velocity=15.89 -> lower=-2.77507351067 upper=-0.645771823238 effort=55 velocity=16
- joint FL_hip_joint: limit lower=-1.2217304763960306 upper=1.2217304763960306 effort=35.278 velocity=20 -> lower=-1.2217304764 upper=1.2217304764 effort=44 velocity=20; origin xyz=0.2407 0.051 0 rpy=0 0 0 -> xyz=0.2399 0.051 0 rpy=0 0 0
- joint FL_thigh_joint: limit effort=35.278 velocity=20 -> lower=-1.0471975512 upper=4.18879020479 effort=44 velocity=20; origin xyz=0 0.0868 0 rpy=0 0 0 -> xyz=0 0.083 0 rpy=0 0 0; type continuous -> revolute
- joint FR_calf_joint: limit lower=-2.775073510670984 upper=-0.6457718232379019 effort=44.4 velocity=15.89 -> lower=-2.77507351067 upper=-0.645771823238 effort=55 velocity=16
- joint FR_hip_joint: limit lower=-1.2217304763960306 upper=1.2217304763960306 effort=35.278 velocity=20 -> lower=-1.2217304764 upper=1.2217304764 effort=44 velocity=20; origin xyz=0.2407 -0.051 0 rpy=0 0 0 -> xyz=0.2399 -0.051 0 rpy=0 0 0
- joint FR_thigh_joint: limit effort=35.278 velocity=20 -> lower=-1.0471975512 upper=4.18879020479 effort=44 velocity=20; origin xyz=0 -0.0868 0 rpy=0 0 0 -> xyz=0 -0.083 0 rpy=0 0 0; type continuous -> revolute
- joint RL_calf_joint: limit lower=-2.775073510670984 upper=-0.6457718232379019 effort=44.4 velocity=15.89 -> lower=-2.77507351067 upper=-0.645771823238 effort=55 velocity=16
- joint RL_hip_joint: limit lower=-1.2217304763960306 upper=1.2217304763960306 effort=35.278 velocity=20 -> lower=-1.2217304764 upper=1.2217304764 effort=44 velocity=20; origin xyz=-0.2407 0.051 0 rpy=0 0 0 -> xyz=-0.2399 0.051 0 rpy=0 0 0
- joint RL_thigh_joint: limit effort=35.278 velocity=20 -> lower=-1.0471975512 upper=4.18879020479 effort=44 velocity=20; origin xyz=0 0.0868 0 rpy=0 0 0 -> xyz=0 0.083 0 rpy=0 0 0; type continuous -> revolute
- joint RR_calf_joint: limit lower=-2.775073510670984 upper=-0.6457718232379019 effort=44.4 velocity=15.89 -> lower=-2.77507351067 upper=-0.645771823238 effort=55 velocity=16
- joint RR_hip_joint: limit lower=-1.2217304763960306 upper=1.2217304763960306 effort=35.278 velocity=20 -> lower=-1.2217304764 upper=1.2217304764 effort=44 velocity=20; origin xyz=-0.2407 -0.051 0 rpy=0 0 0 -> xyz=-0.2399 -0.051 0 rpy=0 0 0
- joint RR_thigh_joint: limit effort=35.278 velocity=20 -> lower=-1.0471975512 upper=4.18879020479 effort=44 velocity=20; origin xyz=0 -0.0868 0 rpy=0 0 0 -> xyz=0 -0.083 0 rpy=0 0 0; type continuous -> revolute

File: robots/aliengo_description/xacro/gazebo.xacro (robot description, xacro)
@@ -8,6 +8,17 @@
         </plugin>
     </gazebo>
+    <gazebo>
+        <plugin name="p3d" filename="libgazebo_ros_p3d.so">
+            <always_on>true</always_on>
+            <update_rate>200</update_rate>
+            <bodyName>base</bodyName>
+            <topicName>/torso_odom</topicName>
+            <frameName>world</frameName>
+            <xyzOffset>0 0 0</xyzOffset>
+            <rpyOffset>0 0 0</rpyOffset>
+        </plugin>
+    </gazebo>
     <!-- Show the trajectory of trunk center. -->
-    <gazebo>
+    <!-- <gazebo>
         <plugin name="3dplot" filename="libLinkPlot3DPlugin.so">
             <frequency>10</frequency>
@@ -19,5 +30,5 @@
         </plugin>
     </gazebo>
-    <!-- Show the trajectory of foot. You can add another trajectory about another foot. -->
+    <- Show the trajectory of foot. You can add another trajectory about another foot. -->
     <!-- <gazebo>
         <plugin name="3dplot" filename="libLinkPlot3DPlugin.so">
