Commit message: change xacro formant of arcdog

File: robots/arclab_robot_description/robots/quadrupedal_robot/common/gazebo.xacro (robot description, xacro)
@@ -2,12 +2,19 @@
 <robot>
     <!-- ros_control plugin -->
-    <gazebo>
+    <!-- <gazebo>
         <plugin name="gazebo_ros_control" filename="libarcdog_hw_sim.so">
-            <robotNamespace>/</robotNamespace>
+            <robotNamespace>/arclab_robot_gazebo</robotNamespace>
             <robotParam>legged_robot_description</robotParam>
             <robotSimType>arcdog_sim/ArcdogHWSim</robotSimType>
         </plugin>
-    </gazebo>
+    </gazebo> -->
+    <!-- ros_control plugin -->
     <gazebo>
+        <plugin name="gazebo_ros_control" filename="libgazebo_ros_control.so">
+            <robotNamespace>/arclab_robot_gazebo</robotNamespace>
+            <robotSimType>gazebo_ros_control/DefaultRobotHWSim</robotSimType>
+        </plugin>
+    </gazebo>
+    <!-- <gazebo>
         <plugin name="p3d_base_controller" filename="libgazebo_ros_p3d.so">
             <alwaysOn>true</alwaysOn>
@@ -20,4 +27,359 @@
             <rpyOffsets>0 0 0</rpyOffsets>
         </plugin>
+    </gazebo> -->
+   <!-- simulate a body pose sensor -->
+    <gazebo>
+        <plugin name="p3d" filename="libgazebo_ros_p3d.so">
+        <alwaysOn>true</alwaysOn>
+        <updateRate>100.0</updateRate>
+        <bodyName>base</bodyName>
+        <topicName>body_pose_ground_truth</topicName>
+        <frameName>world</frameName>
+        <xyzOffsets>0 0 0.0</xyzOffsets>
+        <rpyOffsets>0 0 0.0</rpyOffsets>
+        </plugin>
+    </gazebo>
+    <gazebo>
+        <plugin name="p3d" filename="libgazebo_ros_p3d.so">
+            <always_on>true</always_on>
+            <update_rate>200</update_rate>
+            <bodyName>base</bodyName>
+            <topicName>/torso_odom</topicName>
+            <frameName>world</frameName>
+            <xyzOffset>0 0 0</xyzOffset>
+            <rpyOffset>0 0 0</rpyOffset>
+        </plugin>
+    </gazebo>
+    <!-- Show the trajectory of trunk center. -->
+    <gazebo>
+        <plugin filename="libgazebo_ros_force.so" name="gazebo_ros_force">
+            <bodyName>trunk</bodyName>
+            <topicName>/apply_force/trunk</topicName>
+        </plugin>
+    </gazebo>
+    <gazebo reference="imu_link">
+        <gravity>true</gravity>
+        <sensor name="imu_sensor" type="imu">
+            <always_on>true</always_on>
+            <update_rate>400</update_rate>
+            <visualize>true</visualize>
+            <topic>__default_topic__</topic>
+            <plugin filename="libgazebo_ros_imu_sensor.so" name="imu_plugin">
+                <topicName>trunk_imu</topicName>
+                <bodyName>imu_link</bodyName>
+                <updateRateHZ>400.0</updateRateHZ>
+                <gaussianNoise>0.001</gaussianNoise>
+                <xyzOffset>0 0 0</xyzOffset>
+                <rpyOffset>0 0 0</rpyOffset>
+                <frameName>imu_link</frameName>
+            </plugin>
+            <pose>0 0 0 0 0 0</pose>
+        </sensor>
+    </gazebo>
+    <!-- Depth camera -->
+    <!-- <gazebo>
+        <plugin name="camera_plugin" filename="libgazebo_ros_openni_kinect.so">
+            <baseline>0.025</baseline>
+            <always_on>true</always_on>
+            <updateRate>0.0</updateRate>
+            <cameraName>unitree_camera_left</cameraName>
+            <frameName>depthCamera_link_left</frameName>
+            <imageTopicName>rgb/imageRaw_left</imageTopicName>
+            <depthImageTopicName>depth/imageRaw_left</depthImageTopicName>
+            <pointCloudTopicName>depth/points_left</pointCloudTopicName>
+            <cameraInfoTopicName>rgb/cameraInfo_left</cameraInfoTopicName>
+            <depthImageCameraInfoTopicName>depth/cameraInfo_left</depthImageCameraInfoTopicName>
+            <pointCloudCutoff>0.1</pointCloudCutoff>
+            <pointCloudCutoffMax>1.5</pointCloudCutoffMax>
+            <distortionK1>0.0</distortionK1>
+            <distortionK2>0.0</distortionK2>
+            <distortionK3>0.0</distortionK3>
+            <distortionT1>0.0</distortionT1>
+            <distortionT2>0.0</distortionT2>
+            <CxPrime>0.0</CxPrime>
+            <Cx>0.0045</Cx>
+            <Cy>0.0039</Cy>
+            <focalLength>0.004</focalLength>
+            <hackBaseline>0.0</hackBaseline>
+        </plugin>
+    </gazebo> -->
+    <!-- <gazebo reference="depthCamera_link_left">
+        <sensor name="unitree_camera_left" type="depth_camera">
+            <update_rate>16</update_rate>
+            <always_on>true</always_on>
+            <visualize>true</visualize>
+            <camera>
+                <horizontal_fov>2.094</horizontal_fov>
+                <image>
+                    <width>928</width>
+                    <height>800</height>
+                    <format>R8G8B8</format>
+                </image>
+                <depth_camera></depth_camera>
+                <clip>
+                    <near>0.1</near>
+                    <far>100</far>
+                </clip>
+            </camera>
+            <plugin name="camera_plugin" filename="libgazebo_ros_openni_kinect.so">
+                <baseline>0.025</baseline>
+                <always_on>true</always_on>
+                <updateRate>0.0</updateRate>
+                <cameraName>unitree_camera_left</cameraName>
+                <frameName>depthCamera_link_left</frameName>
+                <imageTopicName>rgb/imageRaw_left</imageTopicName>
+                <depthImageTopicName>depth/imageRaw_left</depthImageTopicName>
+                <pointCloudTopicName>depth/points_left</pointCloudTopicName>
+                <cameraInfoTopicName>rgb/cameraInfo_left</cameraInfoTopicName>
+                <depthImageCameraInfoTopicName>depth/cameraInfo_left</depthImageCameraInfoTopicName>
+                <pointCloudCutoff>0.1</pointCloudCutoff>
+                <pointCloudCutoffMax>1.5</pointCloudCutoffMax>
+                <distortionK1>0.0</distortionK1>
+                <distortionK2>0.0</distortionK2>
+                <distortionK3>0.0</distortionK3>
+                <distortionT1>0.0</distortionT1>
+                <distortionT2>0.0</distortionT2>
+                <CxPrime>0.0</CxPrime>
+                <Cx>0.0045</Cx>
+                <Cy>0.0039</Cy>
+                <focalLength>0.004</focalLength>
+                <hackBaseline>0.0</hackBaseline>
+            </plugin>
+        </sensor>
+    </gazebo> -->
+  <gazebo reference="depthCamera_link_left">
+    <sensor name="camera_link_camera" type="depth">
+      <update_rate>20</update_rate>
+      <camera>
+        <horizontal_fov>1.047198</horizontal_fov>
+        <image>
+          <width>640</width>
+          <height>480</height>
+          <format>R8G8B8</format>
+        </image>
+        <clip>
+          <near>0.05</near>
+          <far>3</far>
+        </clip>
+      </camera>
+      <plugin name="camera_link_controller" filename="libgazebo_ros_openni_kinect.so">
+        <baseline>0.2</baseline>
+        <alwaysOn>true</alwaysOn>
+        <updateRate>1.0</updateRate>
+        <cameraName>camera_link_ir</cameraName>
+        <imageTopicName>/camera_link/color/image_raw</imageTopicName>
+        <cameraInfoTopicName>/camera_link/color/camera_info</cameraInfoTopicName>
+        <depthImageTopicName>/camera_link/depth/image_raw</depthImageTopicName>
+        <depthImageInfoTopicName>/camera_link/depth/camera_info</depthImageInfoTopicName>
+        <pointCloudTopicName>/camera_link/depth/points</pointCloudTopicName>
+        <frameName>depthCamera_link_left</frameName>
+        <pointCloudCutoff>0.5</pointCloudCutoff>
+        <pointCloudCutoffMax>3.0</pointCloudCutoffMax>
+        <distortionK1>0.00000001</distortionK1>
+        <distortionK2>0.00000001</distortionK2>
+        <distortionK3>0.00000001</distortionK3>
+        <distortionT1>0.00000001</distortionT1>
+        <distortionT2>0.00000001</distortionT2>
+        <CxPrime>0</CxPrime>
+        <Cx>0</Cx>
+        <Cy>0</Cy>
+        <focalLength>0</focalLength>
+        <hackBaseline>0</hackBaseline>
+      </plugin>
+    </sensor>
+  </gazebo>
+    <!-- Foot contacts. -->
+    <gazebo reference="FR_calf">
+        <sensor name="FR_foot_contact" type="contact">
+        <update_rate>100</update_rate>
+        <plugin name="contactPlugin" filename="libunitreeFootContactPlugin.so"/>
+        <contact>
+            <collision>FR_calf_fixed_joint_lump__FR_foot_collision_1</collision>
+        </contact>
+        </sensor>
+    </gazebo>
+    <gazebo reference="FL_calf">
+        <sensor name="FL_foot_contact" type="contact">
+        <update_rate>100</update_rate>
+        <plugin name="contactPlugin" filename="libunitreeFootContactPlugin.so"/>
+        <contact>
+            <collision>FL_calf_fixed_joint_lump__FL_foot_collision_1</collision>
+        </contact>
+        </sensor>
+    </gazebo>
+    <gazebo reference="RR_calf">
+        <sensor name="RR_foot_contact" type="contact">
+        <update_rate>100</update_rate>
+        <plugin name="contactPlugin" filename="libunitreeFootContactPlugin.so"/>
+        <contact>
+            <collision>RR_calf_fixed_joint_lump__RR_foot_collision_1</collision>
+        </contact>
+        </sensor>
+    </gazebo>
+    <gazebo reference="RL_calf">
+        <sensor name="RL_foot_contact" type="contact">
+        <update_rate>100</update_rate>
+        <plugin name="contactPlugin" filename="libunitreeFootContactPlugin.so"/>
+        <contact>
+            <collision>RL_calf_fixed_joint_lump__RL_foot_collision_1</collision>
+        </contact>
+        </sensor>
+    </gazebo>
+    <!-- Visualization of Foot contacts. -->
+    <gazebo reference="FR_foot">
+        <visual>
+            <plugin name="drawForcePlugin" filename="libunitreeDrawForcePlugin.so">
+                <topicName>FR_foot_contact</topicName>
+            </plugin>
+        </visual>
+    </gazebo>
+    <gazebo reference="FL_foot">
+        <visual>
+            <plugin name="drawForcePlugin" filename="libunitreeDrawForcePlugin.so">
+                <topicName>FL_foot_contact</topicName>
+            </plugin>
+        </visual>
+    </gazebo>
+    <gazebo reference="RR_foot">
+        <visual>
+            <plugin name="drawForcePlugin" filename="libunitreeDrawForcePlugin.so">
+                <topicName>RR_foot_contact</topicName>
+            </plugin>
+        </visual>
+    </gazebo>
+    <gazebo reference="RL_foot">
+        <visual>
+            <plugin name="drawForcePlugin" filename="libunitreeDrawForcePlugin.so">
+                <topicName>RL_foot_contact</topicName>
+            </plugin>
+        </visual>
+    </gazebo>
+    <gazebo reference="base">
+        <material>Gazebo/Green</material>
+        <turnGravityOff>false</turnGravityOff>
+    </gazebo>
+    <gazebo reference="trunk">
+        <mu1>0.2</mu1>
+        <mu2>0.2</mu2>
+        <kp  value="1000000.0"/>
+        <kd  value="1.0"/>
+    </gazebo>
+    <gazebo reference="stick_link">
+        <mu1>0.2</mu1>
+        <mu2>0.2</mu2>
+        <material>Gazebo/White</material>
+    </gazebo>
+    <gazebo reference="imu_link">
+        <mu1>0.2</mu1>
+        <mu2>0.2</mu2>
+        <material>Gazebo/Red</material>
+    </gazebo>
+    <!-- FL leg -->
+    <gazebo reference="FL_hip">
+        <mu1>0.2</mu1>
+        <mu2>0.2</mu2>
+        <material>Gazebo/DarkGrey</material>
+    </gazebo>
+    <gazebo reference="FL_thigh">
+        <mu1>0.2</mu1>
+        <mu2>0.2</mu2>
+        <self_collide>1</self_collide>
+        <material>Gazebo/DarkGrey</material>
+        <kp  value="1000000.0"/>
+        <kd  value="1.0"/>
+    </gazebo>
+    <gazebo reference="FL_calf">
+        <mu1>0.2</mu1>
+        <mu2>0.2</mu2>
+        <self_collide>1</self_collide>
+    </gazebo>
+    <gazebo reference="FL_foot">
+        <mu1>0.6</mu1>
+        <mu2>0.6</mu2>
+        <self_collide>1</self_collide>
+        <material>Gazebo/DarkGrey</material>
+        <kp  value="1000000.0"/>
+        <kd  value="1.0"/>
+    </gazebo>
+    <!-- FR leg -->
+    <gazebo reference="FR_hip">
+        <mu1>0.2</mu1>
+        <mu2>0.2</mu2>
+        <material>Gazebo/DarkGrey</material>
+    </gazebo>
+    <gazebo reference="FR_thigh">
+        <mu1>0.2</mu1>
+        <mu2>0.2</mu2>
+        <self_collide>1</self_collide>
+        <material>Gazebo/DarkGrey</material>
+        <kp  value="1000000.0"/>
+        <kd  value="1.0"/>
+    </gazebo>
+    <gazebo reference="FR_calf">
+        <mu1>0.2</mu1>
+        <mu2>0.2</mu2>
+        <self_collide>1</self_collide>
+    </gazebo>
+    <gazebo reference="FR_foot">
+        <mu1>0.6</mu1>
+        <mu2>0.6</mu2>
+        <self_collide>1</self_collide>
+        <material>Gazebo/DarkGrey</material>
+        <kp  value="1000000.0"/>
+        <kd  value="1.0"/>
+    </gazebo>
+    <!-- RL leg -->
+    <gazebo reference="RL_hip">
+        <mu1>0.2</mu1>
+        <mu2>0.2</mu2>
+        <material>Gazebo/DarkGrey</material>
+    </gazebo>
+    <gazebo reference="RL_thigh">
+        <mu1>0.2</mu1>
+        <mu2>0.2</mu2>
+        <self_collide>1</self_collide>
+        <material>Gazebo/DarkGrey</material>
+        <kp  value="1000000.0"/>
+        <kd  value="1.0"/>
+    </gazebo>
+    <gazebo reference="RL_calf">
+        <mu1>0.2</mu1>
+        <mu2>0.2</mu2>
+        <self_collide>1</self_collide>
+    </gazebo>
+    <gazebo reference="RL_foot">
+        <mu1>0.6</mu1>
+        <mu2>0.6</mu2>
+        <self_collide>1</self_collide>
+        <material>Gazebo/DarkGrey</material>
+        <kp  value="1000000.0"/>
+        <kd  value="1.0"/>
+    </gazebo>
+    <!-- RR leg -->
+    <gazebo reference="RR_hip">
+        <mu1>0.2</mu1>
+        <mu2>0.2</mu2>
+        <material>Gazebo/DarkGrey</material>
+    </gazebo>
+    <gazebo reference="RR_thigh">
+        <mu1>0.2</mu1>
+        <mu2>0.2</mu2>
+        <self_collide>1</self_collide>
+        <material>Gazebo/DarkGrey</material>
+        <kp  value="1000000.0"/>
+        <kd  value="1.0"/>
+    </gazebo>
+    <gazebo reference="RR_calf">
+        <mu1>0.2</mu1>
+        <mu2>0.2</mu2>
+        <self_collide>1</self_collide>
+    </gazebo>
+    <gazebo reference="RR_foot">
+        <mu1>0.6</mu1>
+        <mu2>0.6</mu2>
+        <self_collide>1</self_collide>
+        <material>Gazebo/DarkGrey</material>
+        <kp  value="1000000.0"/>
+        <kd  value="1.0"/>
     </gazebo>
 </robot>

File: robots/arclab_robot_description/robots/quadrupedal_robot/common/leg.xacro (robot description, xacro)
@@ -4,5 +4,5 @@
     <xacro:macro name="leg" params="prefix mirror mirror_dae front_hind front_hind_dae simulator *origin">
         <xacro:if value="${simulator == 'ocs2'}">
-            <joint name="${prefix}_HAA" type="revolute">
+            <joint name="${prefix}_hip_joint" type="revolute">
                 <xacro:insert_block name="origin"/>
                 <parent link="base"/>
@@ -73,5 +73,5 @@
         </link>
         <xacro:if value="${simulator == 'ocs2'}">
-            <joint name="${prefix}_HFE" type="revolute">
+            <joint name="${prefix}_though_joint" type="revolute">
                 <origin rpy="0 0 0" xyz="0 ${thigh_offset*mirror} 0"/>
                 <parent link="${prefix}_hip"/>
@@ -131,5 +131,5 @@
         </link>
         <xacro:if value="${simulator == 'ocs2'}">
-            <joint name="${prefix}_KFE" type="revolute">
+            <joint name="${prefix}_calf_joint" type="revolute">
                 <origin rpy="0 0 0" xyz="0 0 ${-thigh_length}"/>
                 <parent link="${prefix}_thigh"/>

File: robots/arclab_robot_description/robots/quadrupedal_robot/common/transmission.xacro (robot description, xacro)
@@ -4,5 +4,5 @@
         <transmission name="${prefix}_HAA_tran">
             <type>transmission_interface/SimpleTransmission</type>
-            <joint name="${prefix}_HAA">
+            <joint name="${prefix}_hip_joint">
                 <hardwareInterface>hardware_interface/EffortJointInterface</hardwareInterface>
             </joint>
@@ -14,5 +14,5 @@
         <transmission name="${prefix}_HFE_tran">
             <type>transmission_interface/SimpleTransmission</type>
-            <joint name="${prefix}_HFE">
+            <joint name="${prefix}_thigh_joint">
                 <hardwareInterface>hardware_interface/EffortJointInterface</hardwareInterface>
             </joint>
@@ -24,5 +24,5 @@
         <transmission name="${prefix}_KFE_tran">
             <type>transmission_interface/SimpleTransmission</type>
-            <joint name="${prefix}_KFE">
+            <joint name="${prefix}_calf_joint">
                 <hardwareInterface>hardware_interface/EffortJointInterface</hardwareInterface>
             </joint>

File: robots/arclab_robot_description/urdf/quadrupedal_robot/arcdog/arcdog_ocs2.urdf (robot description, URDF)
Before this commit: robot robot, 18 links, 17 joints
Joints:
- removed joint FL_HAA
- removed joint FL_HFE
- removed joint FL_KFE
- removed joint FR_HAA
- removed joint FR_HFE
- removed joint FR_KFE
- removed joint RL_HAA
- removed joint RL_HFE
- removed joint RL_KFE
- removed joint RR_HAA
- removed joint RR_HFE
- removed joint RR_KFE
- added joint FL_calf_joint: type revolute, parent FL_thigh, child FL_calf, origin xyz=0 0 -0.2445 rpy=0 0 0, axis 0 1 0, limit lower=-2.775073510670984 upper=-0.6457718232379019 effort=44.4 velocity=15.89
- added joint FL_hip_joint: type revolute, parent base, child FL_hip, origin xyz=0.2407 0.051 0 rpy=0 0 0, axis 1 0 0, limit lower=-1.2217304763960306 upper=1.2217304763960306 effort=35.278 velocity=20
- added joint FL_though_joint: type revolute, parent FL_hip, child FL_thigh, origin xyz=0 0.0868 0 rpy=0 0 0, axis 0 1 0, limit lower=-0.6457718232379019 upper=0.6457718232379019 effort=35.278 velocity=20
- added joint FR_calf_joint: type revolute, parent FR_thigh, child FR_calf, origin xyz=0 0 -0.2445 rpy=0 0 0, axis 0 1 0, limit lower=-2.775073510670984 upper=-0.6457718232379019 effort=44.4 velocity=15.89
- added joint FR_hip_joint: type revolute, parent base, child FR_hip, origin xyz=0.2407 -0.051 0 rpy=0 0 0, axis 1 0 0, limit lower=-1.2217304763960306 upper=1.2217304763960306 effort=35.278 velocity=20
- added joint FR_though_joint: type revolute, parent FR_hip, child FR_thigh, origin xyz=0 -0.0868 0 rpy=0 0 0, axis 0 1 0, limit lower=-0.6457718232379019 upper=0.6457718232379019 effort=35.278 velocity=20
- added joint RL_calf_joint: type revolute, parent RL_thigh, child RL_calf, origin xyz=0 0 -0.2445 rpy=0 0 0, axis 0 1 0, limit lower=-2.775073510670984 upper=-0.6457718232379019 effort=44.4 velocity=15.89
- added joint RL_hip_joint: type revolute, parent base, child RL_hip, origin xyz=-0.2407 0.051 0 rpy=0 0 0, axis 1 0 0, limit lower=-1.2217304763960306 upper=1.2217304763960306 effort=35.278 velocity=20
- added joint RL_though_joint: type revolute, parent RL_hip, child RL_thigh, origin xyz=0 0.0868 0 rpy=0 0 0, axis 0 1 0, limit lower=-0.6457718232379019 upper=0.6457718232379019 effort=35.278 velocity=20
- added joint RR_calf_joint: type revolute, parent RR_thigh, child RR_calf, origin xyz=0 0 -0.2445 rpy=0 0 0, axis 0 1 0, limit lower=-2.775073510670984 upper=-0.6457718232379019 effort=44.4 velocity=15.89
- added joint RR_hip_joint: type revolute, parent base, child RR_hip, origin xyz=-0.2407 -0.051 0 rpy=0 0 0, axis 1 0 0, limit lower=-1.2217304763960306 upper=1.2217304763960306 effort=35.278 velocity=20
- added joint RR_though_joint: type revolute, parent RR_hip, child RR_thigh, origin xyz=0 -0.0868 0 rpy=0 0 0, axis 0 1 0, limit lower=-0.6457718232379019 upper=0.6457718232379019 effort=35.278 velocity=20
