Commit message: plugins update

File: robots/aliengo_description/xacro/camera_d435.xacro (robot description, xacro)
@@ -37,5 +37,5 @@
           <origin xyz="${realsense_d435_front_to_depth} ${realsense_d435_case_offset_y} 0.0" rpy="${M_PI/2} 0 ${M_PI/2}" />
           <geometry>
-            <mesh filename="package://hector_sensors_description/meshes/intel_realsense_d435/D435.dae" scale="0.001 0.001 0.001" />
+            <mesh filename="package://aliengo_description/meshes/depthCamera.dae" scale="0.001 0.001 0.001" />
           </geometry>
         </visual>

File: robots/aliengo_description/xacro/gazebo.xacro (robot description, xacro)
@@ -9,5 +9,5 @@
     </gazebo>
     <gazebo>
-        <plugin name="p3d" filename="libgazebo_ros_p3d.so">
+        <plugin name="p3d_tf" filename="libgazebo_ros_p3d_tf.so">
             <always_on>true</always_on>
             <update_rate>200</update_rate>
@@ -70,5 +70,7 @@
         <sensor name="FR_foot_contact" type="contact">
         <update_rate>100</update_rate>
-        <plugin name="contactPlugin" filename="libunitreeFootContactPlugin.so"/>
+        <plugin name="contactPlugin" filename="libunitreeFootContactPluginRviz.so">
+            <linkName>FR_foot</linkName>
+        </plugin>
         <contact>
             <collision>FR_calf_fixed_joint_lump__FR_foot_collision_1</collision>
@@ -79,5 +81,7 @@
         <sensor name="FL_foot_contact" type="contact">
         <update_rate>100</update_rate>
-        <plugin name="contactPlugin" filename="libunitreeFootContactPlugin.so"/>
+        <plugin name="contactPlugin" filename="libunitreeFootContactPluginRviz.so">
+            <linkName>FL_foot</linkName>
+        </plugin>
         <contact>
             <collision>FL_calf_fixed_joint_lump__FL_foot_collision_1</collision>
@@ -88,5 +92,7 @@
         <sensor name="RR_foot_contact" type="contact">
         <update_rate>100</update_rate>
-        <plugin name="contactPlugin" filename="libunitreeFootContactPlugin.so"/>
+        <plugin name="contactPlugin" filename="libunitreeFootContactPluginRviz.so">
+            <linkName>RR_foot</linkName>
+        </plugin>
         <contact>
             <collision>RR_calf_fixed_joint_lump__RR_foot_collision_1</collision>
@@ -97,5 +103,7 @@
         <sensor name="RL_foot_contact" type="contact">
         <update_rate>100</update_rate>
-        <plugin name="contactPlugin" filename="libunitreeFootContactPlugin.so"/>
+        <plugin name="contactPlugin" filename="libunitreeFootContactPluginRviz.so">
+            <linkName>RL_foot</linkName>
+        </plugin>
         <contact>
             <collision>RL_calf_fixed_joint_lump__RL_foot_collision_1</collision>

Commit message: add depth camera D435(i)

File: robots/aliengo_description/xacro/camera_d435.xacro (robot description, xacro)
@@ -35,7 +35,7 @@
         </inertial>
 	      <visual>
-          <origin xyz="${realsense_d435_front_to_depth} ${realsense_d435_case_offset_y} 0.0" rpy="${M_PI/2} 0 ${M_PI/2}" />
+          <origin xyz="${realsense_d435_front_to_depth} ${realsense_d435_case_offset_y} 0.0" rpy="-1.57 0 -1.57" />
           <geometry>
-            <mesh filename="package://aliengo_description/meshes/depthCamera.dae" scale="0.001 0.001 0.001" />
+            <mesh filename="package://aliengo_description/meshes/d435.dae" scale="1 1 1" />
           </geometry>
         </visual>
@@ -51,4 +51,10 @@
         <material>Gazebo/Grey</material>
       </gazebo>
+      <joint name="${name}_optical_joint" type="fixed">
+        <origin rpy="-1.57 0 -1.57" xyz="0 0 0"/>
+        <parent link="${name}_link"/>
+        <child link="${name}_optical_frame"/>
+      </joint>
+      <link name="${name}_optical_frame"/>
     </xacro:macro>
     <xacro:macro name="realsense_d435_camera_model_with_mount" params="name parent *origin">
@@ -96,5 +102,5 @@
             <depthImageCameraInfoTopicName>depth/camera_info</depthImageCameraInfoTopicName>
             <pointCloudTopicName>${depth_points_topic}</pointCloudTopicName>
-            <frameName>${name}_${frame_name}_optical_frame</frameName>
+            <frameName>${name}_optical_frame</frameName>
             <!-- Important information about frames: Currently, this plugin only supports simulation of color image and depth image/cloud from a single frame.
             This frame is given in the <gazebo reference=""> tag above and is set to the ${name}_link which coincides with the depth camera frame. The camera axis is the X-axis. ROS requires an optical frame

File: robots/aliengo_description/xacro/gazebo.xacro (robot description, xacro)
@@ -6,4 +6,14 @@
             <robotNamespace>/aliengo_gazebo</robotNamespace>
             <robotSimType>gazebo_ros_control/DefaultRobotHWSim</robotSimType>
+        </plugin>
+    </gazebo>
+    <gazebo>
+        <plugin name="p3d" filename="libgazebo_ros_p3d.so">
+            <always_on>true</always_on>
+            <update_rate>200</update_rate>
+            <bodyName>base</bodyName>
+            <topicName>/torso_odom</topicName>
+            <xyzOffset>0 0 0</xyzOffset>
+            <rpyOffset>0 0 0</rpyOffset>
         </plugin>
     </gazebo>
@@ -13,5 +23,5 @@
             <update_rate>200</update_rate>
             <bodyName>base</bodyName>
-            <topicName>/torso_odom</topicName>
+            <topicName>/body_pose_ground_truth</topicName>
             <frameName>world</frameName>
             <xyzOffset>0 0 0</xyzOffset>

File: robots/aliengo_description/xacro/robot.xacro (robot description, xacro)
@@ -131,5 +131,5 @@
     </xacro:depthCamera> -->
     <xacro:realsense_d435_camera name ="camera_d435" parent="base">
-        <origin rpy="0 0.785 0" xyz="0.34 0 0" />
+        <origin rpy="0.0 0.0 0.0" xyz="0.34 0 0" />
     </xacro:realsense_d435_camera>
 </robot>
