Commit message: Improved namespace handling in .xacro

File: robots/aliengo_description/xacro/gazebo.xacro (robot description, xacro)
@@ -1,17 +1,21 @@
 <?xml version="1.0"?>
-<robot>
+<robot xmlns:xacro="http://www.ros.org/wiki/xacro">
     <!-- ros_control plugin -->
+    <xacro:arg name="robot_ns" default="/"/>
     <gazebo>
         <plugin name="gazebo_ros_control" filename="libgazebo_ros_control.so">
-            <robotNamespace>/aliengo_gazebo</robotNamespace>
+            <!-- <robotNamespace>/robot2/aliengo_gazebo</robotNamespace> -->
+            <robotNamespace>${robot_ns}/aliengo_gazebo</robotNamespace>
             <robotSimType>gazebo_ros_control/DefaultRobotHWSim</robotSimType>
+            <robotParam>${robot_ns}/robot_description</robotParam>
         </plugin>
     </gazebo>
     <gazebo>
         <plugin name="p3d" filename="libgazebo_ros_p3d.so">
+            <!-- <robotNamespace>${robot_ns}_aliengo_gazebo</robotNamespace> -->
             <always_on>true</always_on>
             <update_rate>200</update_rate>
             <bodyName>base</bodyName>
-            <topicName>/torso_odom</topicName>
+            <topicName>torso_odom</topicName>
             <frameName>world</frameName>
             <xyzOffset>0 0 0</xyzOffset>

File: robots/aliengo_description/xacro/robot.xacro (robot description, xacro)
@@ -1,4 +1,5 @@
 <?xml version="1.0"?>
 <robot name="aliengo_description" xmlns:xacro="http://www.ros.org/wiki/xacro">
+    <xacro:property name="robot_ns" value="$(arg robot_ns)"/>
     <xacro:include filename="$(find aliengo_description)/xacro/const.xacro"/>
     <xacro:include filename="$(find aliengo_description)/xacro/materials.xacro"/>

File: robots/go1_description/xacro/gazebo.xacro (robot description, xacro)
@@ -1,9 +1,12 @@
 <?xml version="1.0"?>
-<robot>
+<robot xmlns:xacro="http://www.ros.org/wiki/xacro">
     <!-- ros_control plugin -->
+    <xacro:arg name="robot_ns" default="/"/>
     <gazebo>
         <plugin name="gazebo_ros_control" filename="libgazebo_ros_control.so">
-            <robotNamespace>/go1_gazebo</robotNamespace>
+            <!-- <robotNamespace>/robot1/go1_gazebo</robotNamespace> -->
+            <robotNamespace>${robot_ns}/go1_gazebo</robotNamespace>
             <robotSimType>gazebo_ros_control/DefaultRobotHWSim</robotSimType>
+            <robotParam>${robot_ns}/robot_description</robotParam>
         </plugin>
     </gazebo>
@@ -25,5 +28,5 @@
             <update_rate>200</update_rate>
             <bodyName>base</bodyName>
-            <topicName>/torso_odom</topicName>
+            <topicName>torso_odom</topicName>
             <frameName>world</frameName>
             <xyzOffset>0 0 0</xyzOffset>

File: robots/go1_description/xacro/robot.xacro (robot description, xacro)
@@ -1,4 +1,5 @@
 <?xml version="1.0"?>
 <robot name="go1_description" xmlns:xacro="http://www.ros.org/wiki/xacro">
+    <xacro:property name="robot_ns" value="$(arg robot_ns)"/>
     <xacro:include filename="$(find go1_description)/xacro/const.xacro"/>
     <xacro:include filename="$(find go1_description)/xacro/materials.xacro"/>
