Commit message: refactor aliengo, add depth camera on aliengo

File: robots/aliengo_description/xacro/robot.xacro (robot description, xacro)
@@ -5,4 +5,5 @@
     <xacro:include filename="$(find aliengo_description)/xacro/leg.xacro"/>
     <xacro:include filename="$(find aliengo_description)/xacro/gazebo.xacro"/>
+    <xacro:include filename="$(find aliengo_description)/xacro/depthCamera.xacro"/>
     <!-- Rollover Protection mode will add an additional stick on the top, use "true" or "false" to switch it. -->
     <xacro:property name="rolloverProtection" value="false"/>
@@ -125,3 +126,6 @@
     </xacro:leg>
     <!-- <xacro:stairs stairs="15" xpos="0" ypos="2.0" zpos="0" /> -->
+    <xacro:depthCamera camID="1" name="face">
+        <origin rpy="${PI} 0 0" xyz="0.2785 0.0125 0.0167"/>
+    </xacro:depthCamera>
 </robot>

Commit message: add aliengo rl rviz, add a new ground; add d435 depth camera

File: robots/aliengo_description/xacro/robot.xacro (robot description, xacro)
@@ -6,4 +6,5 @@
     <xacro:include filename="$(find aliengo_description)/xacro/gazebo.xacro"/>
     <xacro:include filename="$(find aliengo_description)/xacro/depthCamera.xacro"/>
+    <xacro:include filename="$(find aliengo_description)/xacro/camera_d435.xacro" />
     <!-- Rollover Protection mode will add an additional stick on the top, use "true" or "false" to switch it. -->
     <xacro:property name="rolloverProtection" value="false"/>
@@ -126,6 +127,9 @@
     </xacro:leg>
     <!-- <xacro:stairs stairs="15" xpos="0" ypos="2.0" zpos="0" /> -->
-    <xacro:depthCamera camID="1" name="face">
+    <!-- <xacro:depthCamera camID="1" name="face">
         <origin rpy="${PI} 0 0" xyz="0.2785 0.0125 0.0167"/>
-    </xacro:depthCamera>
+    </xacro:depthCamera> -->
+    <xacro:realsense_d435_camera name ="camera_d435" parent="base">
+        <origin rpy="0 0.785 0" xyz="0.34 0 0" />
+    </xacro:realsense_d435_camera>
 </robot>

Commit message: fix camera bug

File: robots/aliengo_description/xacro/robot.xacro (robot description, xacro)
@@ -132,5 +132,5 @@
     </xacro:depthCamera> -->
     <xacro:realsense_d435_camera name ="camera_d435" parent="base">
-        <origin rpy="0 0.785 0" xyz="0.34 0 0" />
+        <origin rpy="0 0 0" xyz="0.34 0 0" />
     </xacro:realsense_d435_camera>
 </robot>

Commit message: Added Realsense_d435 support to robots and adjusted trunk collision

File: robots/aliengo_description/xacro/robot.xacro (robot description, xacro)
@@ -40,16 +40,16 @@
             <material name="orange"/>
         </visual>
-        <collision>
+        <!-- <collision>
             <origin rpy="0 0 0" xyz="0 0 0"/>
             <geometry>
                 <box size="${trunk_length} ${trunk_width} ${trunk_height}"/>
             </geometry>
-        </collision>
-        <!-- <collision>
+        </collision> -->
+        <collision>
             <origin rpy="0 0 0" xyz="0 0 0"/>
             <geometry>
                 <mesh filename="package://aliengo_description/meshes/trunk.dae" scale="1 1 1"/>
             </geometry>
-        </collision> -->
+        </collision>
         <inertial>
             <origin rpy="0 0 0" xyz="${trunk_com_x} ${trunk_com_y} ${trunk_com_z}"/>

File: robots/go1_description/xacro/robot.xacro (robot description, xacro)
@@ -10,4 +10,5 @@
     <xacro:include filename="$(find go1_description)/xacro/ultraSound.xacro"/>
     <!-- <xacro:include filename="$(find go1_gazebo)/launch/stairs.urdf.xacro"/> -->
+    <xacro:include filename="$(find go1_description)/xacro/camera_d435.xacro" />
     <!-- <xacro:stairs stairs="15" xpos="0" ypos="0" zpos="0" /> -->
     <!-- Rollover Protection mode will add an additional stick on the top, use "true" or "false" to switch it. -->
@@ -43,8 +44,14 @@
             <!-- <material name="orange"/> -->
         </visual>
+        <!-- <collision>
+            <origin rpy="0 0 0" xyz="0 0 0"/>
+            <geometry>
+                <box size="${trunk_length} ${trunk_width} ${trunk_height}"/>
+            </geometry>
+        </collision> -->
         <collision>
             <origin rpy="0 0 0" xyz="0 0 0"/>
             <geometry>
-                <box size="${trunk_length} ${trunk_width} ${trunk_height}"/>
+                <mesh filename="package://go1_description/meshes/trunk.dae" scale="1 1 1"/>
             </geometry>
         </collision>
@@ -162,3 +169,6 @@
         <origin rpy="0 0 0" xyz="0.2747 0.0 -0.0088"/>
     </xacro:ultraSound>
+    <xacro:realsense_d435_camera name ="camera_d435" parent="base">
+        <origin rpy="0 0 0" xyz="0.268 0.02 0" />
+    </xacro:realsense_d435_camera>
 </robot>
