Commit message: add 0.5kg for aliengo trunk, change friction mu to 1.6

File: robots/aliengo_description/xacro/const.xacro (robot description, xacro)
@@ -43,5 +43,5 @@
     <!-- dynamics inertial value -->
     <!-- trunk -->
-    <xacro:property name="trunk_mass" value="11.041"/>
+    <xacro:property name="trunk_mass" value="11.541"/>
     <xacro:property name="trunk_com_x" value="0.008465"/>
     <xacro:property name="trunk_com_y" value="0.004045"/>

File: robots/aliengo_description/xacro/gazebo.xacro (robot description, xacro)
@@ -172,6 +172,6 @@
     </gazebo>
     <gazebo reference="FL_foot">
-        <mu1>0.6</mu1>
-        <mu2>0.6</mu2>
+        <mu1>1.6</mu1>
+        <mu2>1.6</mu2>
         <self_collide>1</self_collide>
         <material>Gazebo/DarkGrey</material>
@@ -199,6 +199,6 @@
     </gazebo>
     <gazebo reference="FR_foot">
-        <mu1>0.6</mu1>
-        <mu2>0.6</mu2>
+        <mu1>1.6</mu1>
+        <mu2>1.6</mu2>
         <self_collide>1</self_collide>
         <material>Gazebo/DarkGrey</material>
@@ -226,6 +226,6 @@
     </gazebo>
     <gazebo reference="RL_foot">
-        <mu1>0.6</mu1>
-        <mu2>0.6</mu2>
+        <mu1>1.6</mu1>
+        <mu2>1.6</mu2>
         <self_collide>1</self_collide>
         <material>Gazebo/DarkGrey</material>
@@ -253,6 +253,6 @@
     </gazebo>
     <gazebo reference="RR_foot">
-        <mu1>0.6</mu1>
-        <mu2>0.6</mu2>
+        <mu1>1.6</mu1>
+        <mu2>1.6</mu2>
         <self_collide>1</self_collide>
         <material>Gazebo/DarkGrey</material>

File: robots/aliengo_description/xacro/robot.xacro (robot description, xacro)
@@ -5,6 +5,6 @@
     <xacro:include filename="$(find aliengo_description)/xacro/leg.xacro"/>
     <xacro:include filename="$(find aliengo_description)/xacro/gazebo.xacro"/>
-    <xacro:include filename="$(find aliengo_description)/xacro/depthCamera.xacro"/>
-    <xacro:include filename="$(find aliengo_description)/xacro/camera_d435.xacro" />
+    <!-- <xacro:include filename="$(find aliengo_description)/xacro/depthCamera.xacro"/> -->
+    <!-- <xacro:include filename="$(find aliengo_description)/xacro/camera_d435.xacro" /> -->
     <!-- Rollover Protection mode will add an additional stick on the top, use "true" or "false" to switch it. -->
     <xacro:property name="rolloverProtection" value="false"/>
@@ -130,6 +130,6 @@
         <origin rpy="${PI} 0 0" xyz="0.2785 0.0125 0.0167"/>
     </xacro:depthCamera> -->
-    <xacro:realsense_d435_camera name ="camera_d435" parent="base">
+    <!-- <xacro:realsense_d435_camera name ="camera_d435" parent="base">
         <origin rpy="0 0.785 0" xyz="0.34 0 0" />
-    </xacro:realsense_d435_camera>
+    </xacro:realsense_d435_camera> -->
 </robot>
